File: KiCad - MIDI-controller/KiCad - MIDI-controller.kicad_pcb (KiCad board)
At the start: 2 copper layers, 66 parts, among them SW1 SW_Push, SW10 SW_Push, SW11 SW_Push, SW12 SW_Push, SW13 SW_Push, SW14 SW_Push, SW15 SW_Push, SW16 SW_Push, SW17 SW_Push, SW18 SW_Push, SW19 SW_Push, SW2 SW_Push, SW20 SW_Push, SW21 RotaryEncoder_Switch, SW22 RotaryEncoder_Switch, SW23 RotaryEncoder_Switch, SW3 SW_Push, SW4 SW_Push, SW5 SW_Push, SW6 SW_Push, SW7 SW_Push, SW8 SW_Push, SW9 SW_Push, U1 ESP32-S3-WROOM-1, U2 CD74HC4067M, U3 CD74HC4067M

Commit message: Day 5
Parts:
- D1, D10, D11, D12, D13, D14, D15, D16, D17, D18, D19, D2, D20, D3, D4, D5, D6, D7, D8, D9: moved to B.Cu
- RV1, RV10, RV2, RV3, RV4, RV5, RV6, RV7, RV8, RV9: footprint Potentiometer_THT:Potentiometer_Bourns_PTA6043_Single_Slide -> Connector_PinHeader_2.54mm:PinHeader_1x03_P2.54mm_Vertical
- moved RV10 42.1 mm to (220.3, 139.6)
- moved RV3 42.1 mm to (79.3, 139.6)
- moved RV4 42.1 mm to (98.3, 139.6)
- moved RV6 42.1 mm to (136.3, 139.6)
- moved RV7 42.1 mm to (155.3, 139.6)
- moved RV8 42.1 mm to (174.4, 139.6)
- moved RV9 42.1 mm to (193.5, 139.6)
- moved RV1 42.1 mm to (41.1, 139.6)
- moved RV2 42.1 mm to (60.2, 139.6)
- moved RV5 42.1 mm to (117.3, 139.6)
- moved U1 23.0 mm to (245.2, 70.8)
- moved RV13 23.0 mm to (84.8, 81.6)
- moved RV14 23.0 mm to (103.8, 81.6)
- moved RV16 23.0 mm to (141.8, 81.6)
- moved RV17 23.0 mm to (160.8, 81.6)
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Routing:
- net Net-(U2-GND): track 0.00 -> 565.0 mm, vias 0 -> 10
- net Net-(U1-3V3): track 0.00 -> 533.4 mm, vias 0 -> 4
- net /POT8: track 0.00 -> 423.4 mm, vias 0 -> 4
- net /POT7: track 0.00 -> 404.1 mm, vias 0 -> 11
- net /C0l1: track 0.00 -> 327.3 mm
- net /FAD1: track 0.00 -> 256.3 mm, vias 0 -> 4
- net /ROW1: track 0.00 -> 250.2 mm
- net /POT1: track 0.00 -> 245.4 mm, vias 0 -> 2
- net /FAD2: track 0.00 -> 241.4 mm, vias 0 -> 4
- net /ROW2: track 0.00 -> 233.4 mm
- net /FAD3: track 0.00 -> 225.1 mm, vias 0 -> 4
- net /POT2: track 0.00 -> 224.7 mm, vias 0 -> 6
- net /POT3: track 0.00 -> 203.0 mm, vias 0 -> 6
- net /FAD4: track 0.00 -> 195.8 mm, vias 0 -> 2
- net /POT4: track 0.00 -> 183.2 mm, vias 0 -> 5
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Other:
- board outline added: 230 x 112 mm

Commit message: Day 6
Parts:
- moved U1 24.2 mm to (255.2, 48.8)
- moved U3 18.2 mm to (255.3, 80.3), turned to 180 degrees
Routing:
- net Net-(U1-IO38): track 0.00 -> 271.7 mm, vias 0 -> 18
- net /C0L2: track 28.7 -> 276.9 mm, vias 0 -> 28
- net /C0L3: track 29.1 -> 265.2 mm, vias 0 -> 18
- net /C0L4: track 28.5 -> 238.4 mm, vias 0 -> 16
- net Net-(U1-IO39): track 0.00 -> 207.6 mm, vias 0 -> 2
- net /C0L5: track 28.8 -> 223.8 mm, vias 0 -> 18
- net Net-(U1-IO21): track 0.00 -> 186.7 mm, vias 0 -> 10
- net Net-(U2-GND): track 565.0 -> 751.0 mm, vias 10 -> 17
- net Net-(U1-IO41): track 0.00 -> 185.2 mm, vias 0 -> 6
- net Net-(U1-IO40): track 0.00 -> 184.0 mm, vias 0 -> 6
- net /C0L8: track 28.2 -> 207.3 mm, vias 0 -> 19
- net /C0L7: track 28.5 -> 194.4 mm, vias 0 -> 14
- net Net-(U1-IO42): track 0.00 -> 165.8 mm, vias 0 -> 4
- net /POT1: track 245.4 -> 91.7 mm
- net /C0L6: track 28.7 -> 181.5 mm, vias 0 -> 17
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- added copper zone on B.Cu, net Net-(U2-GND)
- added copper zone on F.Cu, net Net-(U2-GND)
Other:
- board size 230 x 112 mm -> 241 x 107.8 mm

Commit message: Day 8
Parts:
- added H1: M3, MountingHole:MountingHole_3.2mm_M3, F.Cu at (35.6, 39.4)
- added H2: M3, MountingHole:MountingHole_3.2mm_M3, F.Cu at (35.4, 139.4)
- added H3: M3, MountingHole:MountingHole_3.2mm_M3, F.Cu at (238.5, 39.5)
- added H4: M3, MountingHole:MountingHole_3.2mm_M3, F.Cu at (268.9, 139.4)
- added H5: M3, MountingHole:MountingHole_3.2mm_M3, F.Cu at (106.5, 42.5)
- added H6: M3, MountingHole:MountingHole_3.2mm_M3, F.Cu at (156.0, 43.8)
- added H7: M3, MountingHole:MountingHole_3.2mm_M3, F.Cu at (129.4, 130.7)
- RV1, RV10, RV2, RV3, RV4, RV5, RV6, RV7, RV8, RV9: value R_Potentiometer -> SC1009G 10k
- RV11, RV12, RV13, RV14, RV15, RV16, RV17, RV18, RV19, RV20: value R_Potentiometer -> RV09 10k
- SW1, SW10, SW11, SW12, SW13, SW14, SW15, SW16, SW17, SW18, SW19, SW2, SW20, SW3, SW4, SW5, SW6, SW7, SW8, SW9: value SW_Push -> Kailh Choc V1; footprint Button_Switch_Keyboard:SW_Cherry_MX_1.00u_Plate -> MIDI-controller:SW_Kailh_Choc_V1_1.00u
- SW21, SW22, SW23: value RotaryEncoder_Switch -> EC11 (THT, switch)
- U1: value ESP32-S3-WROOM-1 -> ESP32-S3 DevKit N16R8; footprint RF_Module:ESP32-S3-WROOM-1 -> MIDI-controller:ESP32-S3-DevKitC-1_44P_W25.4mm
- U2, U3: value CD74HC4067M -> CD4067BE; footprint Package_SO:SOIC-24W_7.5x15.4mm_P1.27mm -> Package_DIP:DIP-24_W15.24mm
- moved U3 63.0 mm to (236.0, 140.3), turned to 90 degrees
- moved U1 46.0 mm to (270.8, 92.1), turned to 180 degrees
- moved U2 11.4 mm to (236.0, 119.0)
- moved SW13 5.68 mm to (82.3, 94.1)
- moved SW3 5.68 mm to (82.3, 114.6)
- moved SW14 5.68 mm to (101.3, 94.1)
- moved SW4 5.68 mm to (101.3, 114.6)
- moved SW15 5.68 mm to (120.3, 94.1)
- moved SW5 5.68 mm to (120.3, 114.6)
- moved SW1 5.68 mm to (44.1, 114.6)
- moved SW11 5.68 mm to (44.1, 94.1)
- moved SW12 5.68 mm to (63.2, 94.1)
- moved SW2 5.68 mm to (63.2, 114.6)
- moved SW10 5.68 mm to (223.3, 114.6)
- moved SW16 5.68 mm to (139.3, 94.1)
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Connections:
- RV1 pad 1: Net-(U1-3V3) -> Net-(U2-VCC)
- RV10 pad 1: Net-(U1-3V3) -> Net-(U2-VCC)
- RV11 pad 1: Net-(U1-3V3) -> Net-(U2-VCC)
- RV12 pad 1: Net-(U1-3V3) -> Net-(U2-VCC)
- RV13 pad 1: Net-(U1-3V3) -> Net-(U2-VCC)
- RV14 pad 1: Net-(U1-3V3) -> Net-(U2-VCC)
- RV15 pad 1: Net-(U1-3V3) -> Net-(U2-VCC)
- RV16 pad 1: Net-(U1-3V3) -> Net-(U2-VCC)
- RV17 pad 1: Net-(U1-3V3) -> Net-(U2-VCC)
- RV18 pad 1: Net-(U1-3V3) -> Net-(U2-VCC)
- RV19 pad 1: Net-(U1-3V3) -> Net-(U2-VCC)
- RV2 pad 1: Net-(U1-3V3) -> Net-(U2-VCC)
- RV20 pad 1: Net-(U1-3V3) -> Net-(U2-VCC)
- RV3 pad 1: Net-(U1-3V3) -> Net-(U2-VCC)
- RV4 pad 1: Net-(U1-3V3) -> Net-(U2-VCC)
- RV5 pad 1: Net-(U1-3V3) -> Net-(U2-VCC)
- RV6 pad 1: Net-(U1-3V3) -> Net-(U2-VCC)
- RV7 pad 1: Net-(U1-3V3) -> Net-(U2-VCC)
- RV8 pad 1: Net-(U1-3V3) -> Net-(U2-VCC)
- RV9 pad 1: Net-(U1-3V3) -> Net-(U2-VCC)
- U1 pad 1: Net-(U2-GND) -> Net-(U2-VCC)
- U1 pad 13: unconnected-(U1-USB_D--Pad13) -> /C0l1
- U1 pad 14: unconnected-(U1-USB_D+-Pad14) -> Net-(U1-IO46)
- U1 pad 15: /C0l1 -> /C0L7
- U1 pad 16: Net-(U1-IO46) -> /C0L8
- U1 pad 17: /C0L7 -> /C0L9
- U1 pad 18: /C0L8 -> /C0L10
- U1 pad 19: /C0L9 -> Net-(U1-IO13)
- U1 pad 2: Net-(U1-3V3) -> Net-(U2-VCC)
- U1 pad 20: /C0L10 -> Net-(U1-IO14)
- U1 pad 21: Net-(U1-IO13) -> unconnected-(U1-5V-Pad21)
- U1 pad 22: Net-(U1-IO14) -> Net-(U2-GND)
- U1 pad 23: Net-(U1-IO21) -> Net-(U2-GND)
- U1 pad 24: Net-(U1-IO47) -> unconnected-(U1-TX-Pad24)
- U1 pad 26: Net-(U1-IO45) -> /ROW1
- U1 pad 27: unconnected-(U1-IO0-Pad27) -> /ROW2
- U1 pad 28: unconnected-(U1-IO35-Pad28) -> Net-(U1-IO42)
- U1 pad 29: unconnected-(U1-IO36-Pad29) -> Net-(U1-IO41)
- U1 pad 30: unconnected-(U1-IO37-Pad30) -> Net-(U1-IO40)
- U1 pad 31: Net-(U1-IO38) -> Net-(U1-IO39)
- U1 pad 32: Net-(U1-IO39) -> Net-(U1-IO38)
- U1 pad 33: Net-(U1-IO40) -> unconnected-(U1-IO37-Pad33)
- U1 pad 34: Net-(U1-IO41) -> unconnected-(U1-IO36-Pad34)
- U1 pad 35: Net-(U1-IO42) -> unconnected-(U1-IO35-Pad35)
- U1 pad 37: unconnected-(U1-TXD0-Pad37) -> Net-(U1-IO45)
- U1 pad 38: /ROW2 -> unconnected-(U1-IO48-Pad38)
- U1 pad 39: /ROW1 -> Net-(U1-IO47)
- U1 pad 40: Net-(U2-GND) -> Net-(U1-IO21)
- U1 pad 41: Net-(U2-GND) -> unconnected-(U1-IO20/USB_D+-Pad41)
- U2 pad 24: Net-(U1-3V3) -> Net-(U2-VCC)
- U3 pad 24: Net-(U1-3V3) -> Net-(U2-VCC)
Routing:
- net Net-(U1-3V3): track 624.8 -> 0.00 mm, vias 13 -> 0
- net Net-(U2-VCC): track 0.00 -> 574.2 mm, vias 0 -> 6
- net /C0L2: track 276.9 -> 471.8 mm, vias 28 -> 39
- net Net-(U2-GND): track 751.0 -> 568.8 mm, vias 17 -> 5
- net /POT1: track 91.7 -> 251.1 mm, vias 2 -> 5
- net /POT2: track 140.4 -> 266.3 mm, vias 6 -> 14
- net /C0L3: track 265.2 -> 367.6 mm, vias 18 -> 24
- net Net-(U1-IO38): track 271.7 -> 174.9 mm, vias 18 -> 6
- net /ROW1: track 384.4 -> 304.0 mm
- net /C0l1: track 451.3 -> 381.7 mm, vias 10 -> 2
- net /FAD5: track 200.7 -> 132.3 mm, vias 6 -> 1
- net /FAD9: track 127.3 -> 59.2 mm, vias 3 -> 1
- net /FAD10: track 100.1 -> 32.2 mm, vias 5 -> 2
- net /ROW2: track 272.9 -> 206.2 mm, vias 10 -> 1
- net /FAD8: track 140.6 -> 75.1 mm, vias 6 -> 3
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