File: KiCad - MIDI-controller/KiCad - MIDI-controller.kicad_sch (KiCad schematic)
At the start: 41 parts, among them SW1 SW_Push, SW10 SW_Push, SW11 SW_Push, SW12 SW_Push, SW13 SW_Push, SW14 SW_Push, SW15 SW_Push, SW16 SW_Push, SW17 SW_Push, SW18 SW_Push, SW19 SW_Push, SW2 SW_Push, SW20 SW_Push, SW3 SW_Push, SW4 SW_Push, SW5 SW_Push, SW6 SW_Push, SW7 SW_Push, SW8 SW_Push, SW9 SW_Push, U1 ESP32-S3-WROOM-1

Commit message: Day 3
Parts:
- added RV1, RV10, RV11, RV12, RV13, RV14, RV15, RV16, RV17, RV18, RV19, RV2, RV20, RV3, RV4, RV5, RV6, RV7, RV8, RV9: R_Potentiometer, Package_SO:TSSOP-20_4.4x6.5mm_P0.65mm, symbol Device:R_Potentiometer
- added SW21, SW22, SW23: RotaryEncoder_Switch, symbol Device:RotaryEncoder_Switch
- added U2, U3: CD74HC4067M, Package_SO:SOIC-24W_7.5x15.4mm_P1.27mm, symbol 74xx:CD74HC4067M
Connections:
- net at U1.1 (GND), U1.40 (GND), U1.41 (GND): now also RV1.3, RV10.3, RV11.3, RV12.3, RV13.3, RV14.3, RV15.3, RV16.3, RV17.3, RV18.3, RV19.3, RV2.3, RV20.3, RV3.3, RV4.3, RV5.3, RV6.3, RV7.3, RV8.3, RV9.3, SW21.C, SW21.S2, SW22.C, SW22.S2, SW23.C, SW23.S2, U2.12 (GND), U2.15 (~{E}), U3.12 (GND), U3.15 (~{E})
- net at U1.10 (IO17): now also U3.1 (COM)
- net at U1.11 (IO18): now also U2.1 (COM)
- net at U1.16 (IO46): now also SW23.B
- net at U1.2 (3V3): now also RV1.1, RV10.1, RV11.1, RV12.1, RV13.1, RV14.1, RV15.1, RV16.1, RV17.1, RV18.1, RV19.1, RV2.1, RV20.1, RV3.1, RV4.1, RV5.1, RV6.1, RV7.1, RV8.1, RV9.1, U2.24 (VCC), U3.24 (VCC)
- net at U1.21 (IO13): now also U2.10 (S0), U3.10 (S0)
- net at U1.22 (IO14): now also U2.11 (S1), U3.11 (S1)
- net at U1.23 (IO21): now also SW21.A
- net at U1.24 (IO47): now also SW23.S1
- net at U1.26 (IO45): now also SW23.A
- net at U1.31 (IO38): now also SW21.B
- net at U1.32 (IO39): now also SW21.S1
- net at U1.33 (IO40): now also SW22.A
- net at U1.34 (IO41): now also SW22.B
- net at U1.35 (IO42): now also SW22.S1
- net at U1.8 (IO15): now also U2.14 (S2), U3.14 (S2)
- net at U1.9 (IO16): now also U2.13 (S3), U3.13 (S3)
- new net FAD1: RV1.2, U3.9 (I0)
- new net FAD10: RV10.2, U3.22 (I9)
- new net FAD2: RV2.2, U3.8 (I1)
- new net FAD3: RV3.2, U3.7 (I2)
- new net FAD4: RV4.2, U3.6 (I3)
- new net FAD5: RV5.2, U3.5 (I4)
- new net FAD6: RV6.2, U3.4 (I5)
- new net FAD7: RV7.2, U3.3 (I6)
- new net FAD8: RV8.2, U3.2 (I7)
- new net FAD9: RV9.2, U3.23 (I8)
- new net POT1: RV11.2, U2.9 (I0)
- new net POT10: RV20.2, U2.22 (I9)
- new net POT2: RV12.2, U2.8 (I1)
- new net POT3: RV13.2, U2.7 (I2)
- new net POT4: RV14.2, U2.6 (I3)
- new net POT5: RV15.2, U2.5 (I4)
- new net POT6: RV16.2, U2.4 (I5)
- new net POT7: RV17.2, U2.3 (I6)
- new net POT8: RV18.2, U2.2 (I7)
- new net POT9: RV19.2, U2.23 (I8)
- no-connect marks 0 -> 22
Other:
- moved on the sheet: D1, D10, D11, D12, D13, D14, D15, D16, D17, D18, D19, D2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

Commit message: Day 4
Parts:
- RV1, RV10, RV2, RV3, RV4, RV5, RV6, RV7, RV8, RV9: footprint Package_SO:TSSOP-20_4.4x6.5mm_P0.65mm -> Potentiometer_THT:Potentiometer_Bourns_PTA6043_Single_Slide
- RV11, RV12, RV13, RV14, RV15, RV16, RV17, RV18, RV19, RV20: footprint Package_SO:TSSOP-20_4.4x6.5mm_P0.65mm -> Potentiometer_THT:Potentiometer_Bourns_PTV09A-1_Single_Vertical
- SW1: footprint Button_Switch_SMD:Nidec_Copal_CAS-120A -> Button_Switch_Keyboard:SW_Cherry_MX_1.00u_Plate
- SW10, SW11, SW12, SW13, SW14, SW15, SW16, SW17, SW18, SW19, SW2, SW20, SW3, SW4, SW5, SW6, SW7, SW8, SW9: footprint (none) -> Button_Switch_Keyboard:SW_Cherry_MX_1.00u_Plate
- SW21, SW22, SW23: footprint (none) -> Rotary_Encoder:RotaryEncoder_Alps_EC11E-Switch_Vertical_H20mm
Changed lines of the file:
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@@
 			)
 		)
-		(property "Footprint" ""
+		(property "Footprint" "Button_Switch_Keyboard:SW_Cherry_MX_1.00u_Plate"
 			(at 71.12 100.33 0)
 			(hide yes)
@@
 			)
 		)
-		(property "Footprint" "Package_SO:TSSOP-20_4.4x6.5mm_P0.65mm"
+		(property "Footprint" "Potentiometer_THT:Potentiometer_Bourns_PTV09A-1_Single_Vertical"
 			(at 374.65 205.74 0)
 			(hide yes)
@@
 			)
 		)
-		(property "Footprint" ""
+		(property "Footprint" "Button_Switch_Keyboard:SW_Cherry_MX_1.00u_Plate"
 			(at 162.56 100.33 0)
 			(hide yes)
@@
 			)
 		)
-		(property "Footprint" ""
+		(property "Footprint" "Button_Switch_Keyboard:SW_Cherry_MX_1.00u_Plate"
 			(at 41.91 100.33 0)
 			(hide yes)
@@
 			)
 		)
-		(property "Footprint" ""
+		(property "Footprint" "Rotary_Encoder:RotaryEncoder_Alps_EC11E-Switch_Vertical_H20mm"
 			(at 57.15 201.676 0)
 			(hide yes)
@@
 			)
 		)
-		(property "Footprint" "Package_SO:TSSOP-20_4.4x6.5mm_P0.65mm"
+		(property "Footprint" "Potentiometer_THT:Potentiometer_Bourns_PTV09A-1_Single_Vertical"
 			(at 303.53 205.74 0)
 			(hide yes)
@@
 			)
 		)
-		(property "Footprint" "Package_SO:TSSOP-20_4.4x6.5mm_P0.65mm"
+		(property "Footprint" "Potentiometer_THT:Potentiometer_Bourns_PTV09A-1_Single_Vertical"
 			(at 334.01 205.74 0)
 			(hide yes)
@@
 			)
 		)
-		(property "Footprint" "Package_SO:TSSOP-20_4.4x6.5mm_P0.65mm"
+		(property "Footprint" "Potentiometer_THT:Potentiometer_Bourns_PTV09A-1_Single_Vertical"
 			(at 364.49 205.74 0)
 			(hide yes)
@@
 			)
 		)
-		(property "Footprint" "Package_SO:TSSOP-20_4.4x6.5mm_P0.65mm"
+		(property "Footprint" "Potentiometer_THT:Potentiometer_Bourns_PTV09A-1_Single_Vertical"
 			(at 354.33 205.74 0)
 			(hide yes)
@@
 			)
 		)
-		(property "Footprint" "Package_SO:TSSOP-20_4.4x6.5mm_P0.65mm"
+		(property "Footprint" "Potentiometer_THT:Potentiometer_Bourns_PTV09A-1_Single_Vertical"
 			(at 344.17 205.74 0)
 			(hide yes)
@@
 			)
 		)
-		(property "Footprint" ""
+		(property "Footprint" "Button_Switch_Keyboard:SW_Cherry_MX_1.00u_Plate"
 			(at 26.67 125.73 0)
 			(hide yes)
@@
 			)
 		)
-		(property "Footprint" ""
+		(property "Footprint" "Rotary_Encoder:RotaryEncoder_Alps_EC11E-Switch_Vertical_H20mm"
 			(at 30.48 201.676 0)
 			(hide yes)
@@
 			)
 		)
-		(property "Footprint" ""
+		(property "Footprint" "Button_Switch_Keyboard:SW_Cherry_MX_1.00u_Plate"
 			(at 147.32 100.33 0)
 			(hide yes)
@@
 			)
 		)
-		(property "Footprint" ""
+		(property "Footprint" "Rotary_Encoder:RotaryEncoder_Alps_EC11E-Switch_Vertical_H20mm"
 			(at 82.55 201.676 0)
 			(hide yes)
@@
 			)
 		)
-		(property "Footprint" "Package_SO:TSSOP-20_4.4x6.5mm_P0.65mm"
+		(property "Footprint" "Potentiometer_THT:Potentiometer_Bourns_PTV09A-1_Single_Vertical"
 			(at 394.97 205.74 0)
 			(hide yes)
@@
 			)
 		)
-		(property "Footprint" "Package_SO:TSSOP-20_4.4x6.5mm_P0.65mm"
+		(property "Footprint" "Potentiometer_THT:Potentiometer_Bourns_PTA6043_Single_Slide"
 			(at 205.74 205.74 0)
 			(hide yes)
@@
 			)
 		)
-		(property "Footprint" ""
+		(property "Footprint" "Button_Switch_Keyboard:SW_Cherry_MX_1.00u_Plate"
 			(at 57.15 125.73 0)
 			(hide yes)
@@
 			)
 		)
-		(property "Footprint" ""
+		(property "Footprint" "Button_Switch_Keyboard:SW_Cherry_MX_1.00u_Plate"
 			(at 102.87 125.73 0)
 			(hide yes)
@@
 			)
 		)
-		(property "Footprint" ""
+		(property "Footprint" "Button_Switch_Keyboard:SW_Cherry_MX_1.00u_Plate"
 			(at 87.63 125.73 0)
 			(hide yes)
@@
 			)
 		)
-		(property "Footprint" ""
+		(property "Footprint" "Button_Switch_Keyboard:SW_Cherry_MX_1.00u_Plate"
 			(at 41.91 125.73 0)
 			(hide yes)
@@
 			)
 		)
-		(property "Footprint" "Button_Switch_SMD:Nidec_Copal_CAS-120A"
+		(property "Footprint" "Button_Switch_Keyboard:SW_Cherry_MX_1.00u_Plate"
 			(at 26.67 100.33 0)
 			(hide yes)
@@
 			)
 		)
-		(property "Footprint" "Package_SO:TSSOP-20_4.4x6.5mm_P0.65mm"
+		(property "Footprint" "Potentiometer_THT:Potentiometer_Bourns_PTA6043_Single_Slide"
 			(at 256.54 205.74 0)
 			(hide yes)
@@
 			)
 		)
-		(property "Footprint" "Package_SO:TSSOP-20_4.4x6.5mm_P0.65mm"
+		(property "Footprint" "Potentiometer_THT:Potentiometer_Bourns_PTV09A-1_Single_Vertical"
 			(at 323.85 205.74 0)
 			(hide yes)
@@
 			)
 		)
-		(property "Footprint" "Package_SO:TSSOP-20_4.4x6.5mm_P0.65mm"
+		(property "Footprint" "Potentiometer_THT:Potentiometer_Bourns_PTA6043_Single_Slide"
 			(at 266.7 205.74 0)
 			(hide yes)
@@
 			)
 		)
-		(property "Footprint" ""
+		(property "Footprint" "Button_Switch_Keyboard:SW_Cherry_MX_1.00u_Plate"
 			(at 163.83 125.73 0)
 			(hide yes)
@@
 			)
 		)
-		(property "Footprint" ""
+		(property "Footprint" "Button_Switch_Keyboard:SW_Cherry_MX_1.00u_Plate"
 			(at 55.88 100.33 0)
 			(hide yes)
@@
 			)
 		)
-		(property "Footprint" ""
+		(property "Footprint" "Button_Switch_Keyboard:SW_Cherry_MX_1.00u_Plate"
 			(at 101.6 100.33 0)
 			(hide yes)
@@
 			)
 		)
-		(property "Footprint" ""
+		(property "Footprint" "Button_Switch_Keyboard:SW_Cherry_MX_1.00u_Plate"
 			(at 72.39 125.73 0)
 			(hide yes)
@@
 			)
 		)
-		(property "Footprint" "Package_SO:TSSOP-20_4.4x6.5mm_P0.65mm"
+		(property "Footprint" "Potentiometer_THT:Potentiometer_Bourns_PTA6043_Single_Slide"
 			(at 236.22 205.74 0)
 			(hide yes)
@@
 			)
 		)
-		(property "Footprint" "Package_SO:TSSOP-20_4.4x6.5mm_P0.65mm"
+		(property "Footprint" "Potentiometer_THT:Potentiometer_Bourns_PTA6043_Single_Slide"
 			(at 215.9 205.74 0)
 			(hide yes)
@@
 			)
 		)
-		(property "Footprint" ""
+		(property "Footprint" "Button_Switch_Keyboard:SW_Cherry_MX_1.00u_Plate"
 			(at 148.59 125.73 0)
 			(hide yes)
@@
 			)
 		)
-		(property "Footprint" ""
+		(property "Footprint" "Button_Switch_Keyboard:SW_Cherry_MX_1.00u_Plate"
 			(at 132.08 100.33 0)
 			(hide yes)
@@
 			)
 		)
-		(property "Footprint" ""
+		(property "Footprint" "Button_Switch_Keyboard:SW_Cherry_MX_1.00u_Plate"
 			(at 116.84 100.33 0)
 			(hide yes)
@@
 			)
 		)
-		(property "Footprint" "Package_SO:TSSOP-20_4.4x6.5mm_P0.65mm"
+		(property "Footprint" "Potentiometer_THT:Potentiometer_Bourns_PTA6043_Single_Slide"
 			(at 226.06 205.74 0)
 			(hide yes)
@@
 			)
 		)
-		(property "Footprint" ""
+		(property "Footprint" "Button_Switch_Keyboard:SW_Cherry_MX_1.00u_Plate"
 			(at 118.11 125.73 0)
 			(hide yes)
@@
 			)
 		)
-		(property "Footprint" "Package_SO:TSSOP-20_4.4x6.5mm_P0.65mm"
+		(property "Footprint" "Potentiometer_THT:Potentiometer_Bourns_PTV09A-1_Single_Vertical"
 			(at 313.69 205.74 0)
 			(hide yes)
@@
 			)
 		)
-		(property "Footprint" "Package_SO:TSSOP-20_4.4x6.5mm_P0.65mm"
+		(property "Footprint" "Potentiometer_THT:Potentiometer_Bourns_PTA6043_Single_Slide"
 			(at 276.86 205.74 0)
 			(hide yes)
@@
 			)
 		)
-		(property "Footprint" ""
+		(property "Footprint" "Button_Switch_Keyboard:SW_Cherry_MX_1.00u_Plate"
 			(at 86.36 100.33 0)
 			(hide yes)
@@
 			)
 		)
-		(property "Footprint" "Package_SO:TSSOP-20_4.4x6.5mm_P0.65mm"
+		(property "Footprint" "Potentiometer_THT:Potentiometer_Bourns_PTA6043_Single_Slide"
 			(at 246.38 205.74 0)
 			(hide yes)
@@
 			)
 		)
-		(property "Footprint" ""
+		(property "Footprint" "Button_Switch_Keyboard:SW_Cherry_MX_1.00u_Plate"
 			(at 133.35 125.73 0)
 			(hide yes)
@@
 			)
 		)
-		(property "Footprint" "Package_SO:TSSOP-20_4.4x6.5mm_P0.65mm"
+		(property "Footprint" "Potentiometer_THT:Potentiometer_Bourns_PTV09A-1_Single_Vertical"
 			(at 384.81 205.74 0)
 			(hide yes)
@@
 			)
 		)
-		(property "Footprint" "Package_SO:TSSOP-20_4.4x6.5mm_P0.65mm"
+		(property "Footprint" "Potentiometer_THT:Potentiometer_Bourns_PTA6043_Single_Slide"
 			(at 195.58 205.74 0)
 			(hide yes)
@@
 			)
 		)
-		(property "Footprint" "Package_SO:TSSOP-20_4.4x6.5mm_P0.65mm"
+		(property "Footprint" "Potentiometer_THT:Potentiometer_Bourns_PTA6043_Single_Slide"
 			(at 185.42 205.74 0)
 			(hide yes)

Commit message: Day 8
Parts:
- RV1, RV10, RV2, RV3, RV4, RV5, RV6, RV7, RV8, RV9: value R_Potentiometer -> SC1009G 10k; footprint Potentiometer_THT:Potentiometer_Bourns_PTA6043_Single_Slide -> Connector_PinHeader_2.54mm:PinHeader_1x03_P2.54mm_Vertical
- RV11, RV12, RV13, RV14, RV15, RV16, RV17, RV18, RV19, RV20: value R_Potentiometer -> RV09 10k
- SW1, SW10, SW11, SW12, SW13, SW14, SW15, SW16, SW17, SW18, SW19, SW2, SW20, SW3, SW4, SW5, SW6, SW7, SW8, SW9: value SW_Push -> Kailh Choc V1; footprint Button_Switch_Keyboard:SW_Cherry_MX_1.00u_Plate -> MIDI-controller:SW_Kailh_Choc_V1_1.00u
- SW21, SW22, SW23: value RotaryEncoder_Switch -> EC11 (THT, switch)
- U1: value ESP32-S3-WROOM-1 -> ESP32-S3 DevKit N16R8; footprint RF_Module:ESP32-S3-WROOM-1 -> MIDI-controller:ESP32-S3-DevKitC-1_44P_W25.4mm; symbol RF_Module:ESP32-S3-WROOM-1 -> MIDI-controller:ESP32-S3-DevKitC-1
- U2, U3: value CD74HC4067M -> CD4067BE; footprint Package_SO:SOIC-24W_7.5x15.4mm_P1.27mm -> Package_DIP:DIP-24_W15.24mm
Connections:
- net C0L10: now also U1.18 (IO12); no longer U1.20 (IO12)
- net C0L7: now also U1.15 (IO9); no longer U1.17 (IO9)
- net C0L8: now also U1.16 (IO10); no longer U1.18 (IO10)
- net C0L9: now also U1.17 (IO11); no longer U1.19 (IO11)
- net C0l1: now also U1.13 (IO3); no longer U1.15 (IO3)
- net ROW1: now also U1.26 (IO1); no longer U1.39 (IO1)
- net ROW2: now also U1.27 (IO2); no longer U1.38 (IO2)
- net at RV1.1, RV10.1, RV11.1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: now also U1.1 (3V3)
- net at RV1.3, RV10.3, RV11.3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: now also U1.22 (GND), U1.23 (GND), U1.43 (GND), U1.44 (GND); no longer U1.1 (GND), U1.40 (GND), U1.41 (GND)
- net at SW22.A: now also U1.30 (IO40); no longer U1.33 (IO40)
- net at SW22.B: now also U1.29 (IO41); no longer U1.34 (IO41)
- net at SW22.S1: now also U1.28 (IO42); no longer U1.35 (IO42)
- net at U1.14 (IO46): now also SW23.B
- net at U2.10 (S0), U3.10 (S0): now also U1.19 (IO13); no longer U1.21 (IO13)
- net at U2.11 (S1), U3.11 (S1): now also U1.20 (IO14); no longer U1.22 (IO14)
- net at SW21.A: now also U1.40 (IO21); no longer U1.23 (IO21)
- net at U1.24 (TX): no longer SW23.S1
- net at SW23.A: now also U1.37 (IO45); no longer U1.26 (IO45)
- net at U1.31 (IO39): now also SW21.S1; no longer SW21.B
- net at U1.32 (IO38): now also SW21.B; no longer SW21.S1
- new net: SW23.S1, U1.39 (IO47)
